File: Power-Board/PowerBoard.kicad_pcb (KiCad board)
At the start: 2 copper layers, 77.5 x 107.9 mm, 64 parts, among them J1 IN1, J10 probe3, J11 Battery_out, J12 Buck_out, J13 IN2, J14 Boost_out, J15 Buck_out, J16 Conn_01x02_Male, J17 Conn_01x02_Male, J18 Battery_out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

Commit message: Added Gerber Files
Other:
- net class Default removed
